File: ecp5_sys_v1/FPGA.kicad_sch (KiCad schematic)
At the start: 0 parts

Commit message: Worked on USB
Parts:
- added C1: 100n, PCM_JLCPCB:C_0402, symbol PCM_JLCPCB-Capacitors:0402,100nF
- added J1: Conn_02x03_Odd_Even, symbol Connector_Generic:Conn_02x03_Odd_Even
- added R1, R2, R3, R4: 10K, PCM_JLCPCB:R_0402, symbol PCM_JLCPCB-Resistors:0402,10kΩ
- added R10, R9: 15K, PCM_JLCPCB:R_0402, symbol PCM_JLCPCB-Resistors:0402,15kΩ
- added R11, R12, R13, R14, R6, R8: 4K7, PCM_JLCPCB:R_0402, symbol PCM_JLCPCB-Resistors:0402,4.7kΩ
- added R5: 1K5, PCM_JLCPCB:R_0402, symbol PCM_JLCPCB-Resistors:0402,1.5kΩ
- added R7: 470, PCM_JLCPCB:R_0402, symbol PCM_JLCPCB-Resistors:0402,470Ω
- added U1: LFE5UM-85F-6BG381x, Package_BGA:Lattice_caBGA-381_17x17mm_Layout20x20_P0.8mm, symbol FPGA_Lattice:LFE5UM-85F-6BG381x
- added U2: W25Q128JVP, Package_SON:WSON-8-1EP_6x5mm_P1.27mm_EP3.4x4.3mm, symbol Memory_Flash:W25Q128JVP
Connections:
- new net: U1.B14 (GND), U1.B7 (GND), U1.C19 (GND), U1.D4 (GND), U1.F13 (GND), U1.F14 (GND), U1.F7 (GND), U1.F8 (GND), U1.G10 (GND), U1.G11 (GND), U1.G12 (GND), U1.G13 (GND), U1.G14 (GND), U1.G15 (GND), U1.G17 (GND), U1.G4 (GND), U1.G6 (GND), U1.G7 (GND), U1.G8 (GND), U1.G9 (GND), U1.H19 (GND), U1.J10 (GND), U1.J11 (GND), U1.J12 (GND), U1.J14 (GND), U1.J2 (GND), U1.J7 (GND), U1.J9 (GND), U1.K10 (GND), U1.K11 (GND), U1.K12 (GND), U1.K14 (GND), U1.K15 (GND), U1.K6 (GND), U1.K7 (GND), U1.K9 (GND), U1.L10 (GND), U1.L11 (GND), U1.L12 (GND), U1.L9 (GND), U1.M10 (GND), U1.M11 (GND), U1.M12 (GND), U1.M14 (GND), U1.M16 (GND), U1.M2 (GND), U1.M7 (GND), U1.M9 (GND), U1.N14 (GND), U1.N15 (GND), U1.N6 (GND), U1.N7 (GND), U1.P11 (GND), U1.P12 (GND), U1.P13 (GND), U1.P14 (GND), U1.P7 (GND), U1.P8 (GND), U1.R19 (GND), U1.U10 (GND), U1.U11 (GND), U1.U12 (GND), U1.U13 (GND), U1.U14 (GND), U1.U7 (GND), U1.U8 (GND), U1.U9 (GND), U1.V12 (GND), U1.V13 (GND), U1.V14 (GND), U1.V15 (GND), U1.V16 (GND), U1.V19 (GND), U1.V20 (GND), U1.V5 (GND), U1.V6 (GND), U1.V7 (GND), U1.V8 (GND), U1.V9 (GND), U1.W12 (GND), U1.W15 (GND), U1.W16 (GND), U1.W19 (GND), U1.W6 (GND), U1.W7 (GND)
- new net: U1.F15 (VCCAUX), U1.F6 (VCCAUX), U1.P15 (VCCAUX), U1.P6 (VCCAUX)
- new net: U1.H10 (VCC), U1.H11 (VCC), U1.H12 (VCC), U1.H13 (VCC), U1.H8 (VCC), U1.H9 (VCC), U1.J13 (VCC), U1.J8 (VCC), U1.K13 (VCC), U1.K8 (VCC), U1.L13 (VCC), U1.L8 (VCC), U1.M13 (VCC), U1.M8 (VCC), U1.N10 (VCC), U1.N11 (VCC), U1.N12 (VCC), U1.N13 (VCC), U1.N8 (VCC), U1.N9 (VCC)
- new net: U1.T15 (VCCA1), U1.U15 (VCCA1)
- new net: U1.T6 (VCCA0), U1.U6 (VCCA0)
- new net: U1.V10 (VCCAUXA0), U1.V11 (VCCAUXA0)
- new net: U1.V17 (VCCAUXA1), U1.V18 (VCCAUXA1)
- new net: U1.F11 (VCCIO1), U1.F12 (VCCIO1)
- new net: U1.H14 (VCCIO2), U1.H15 (VCCIO2), U1.J15 (VCCIO2)
- new net: U1.L14 (VCCIO3), U1.L15 (VCCIO3), U1.M15 (VCCIO3)
- new net: U1.F10 (VCCIO0), U1.F9 (VCCIO0)
- new net: U1.L6 (VCCIO6), U1.L7 (VCCIO6), U1.M6 (VCCIO6)
- new net: U1.P10 (VCCIO8), U1.P9 (VCCIO8)
- new net: U1.H6 (VCCIO7), U1.H7 (VCCIO7), U1.J6 (VCCIO7)
- new net +3V3: C1.1, J1.2 (Pin_2), R1.1, R10.1, R11.1, R12.1, R14.1, R2.1, R3.1, R4.1, R5.1, R6.1, R8.1, R9.1, U1.T4 (CFG_1), U2.8 (VCC)
- new net FLASH_CLK: R5.2, U1.U3 (CCLK), U2.6 (CLK)
- new net FLASH_MISO: R3.2, U1.V2 (PB11A), U2.2 (DO/IO_{1})
- new net FLASH_MOSI: R4.2, U1.W2 (PB11B), U2.5 (DI/IO_{0})
- new net FPGA_DONE: R10.2, U1.Y3 (DONE)
- new net FPGA_INIT: R9.2, U1.V3 (~{INIT})
- new net FPGA_JTAG.~{FT_CTS}: R11.2, U1.V4 (TDO)
- new net FPGA_JTAG.~{FT_DCD}: R14.2, U1.U5 (TMS)
- new net FPGA_JTAG.~{FT_DSR}: R13.1, U1.T5 (TCK)
- new net FPGA_JTAG.~{FT_RI}: R12.2, U1.R5 (TDI)
- new net FPGA_PROGRAM: R7.2, R8.2, U1.W3 (~{PROGRAM})
- new net FPGA_PROGRAM_INIT: R7.1
- new net GND: C1.2, J1.1 (Pin_1), R13.2, U1.R4 (CFG_2), U1.U4 (CFG_0), U2.4 (GND), U2.9 (EP)
- new net TEST_MODE_FPGA_CLK: J1.4 (Pin_4)
- new net TEST_MODE_FPGA_CS: J1.5 (Pin_5)
- new net TEST_MODE_FPGA_MISO: J1.3 (Pin_3)
- new net TEST_MODE_FPGA_MOSI: J1.6 (Pin_6)
- new net ~{FLASH_CS}: R6.2, U1.R2 (PB15A), U2.1 (~{CS})
- new net ~{FLASH_RESET}: R1.2, U1.W1 (PB9A), U2.7 (~{HOLD}/~{RESET}/IO_{3})
- new net ~{FLASH_WP}: R2.2, U1.Y2 (PB9B), U2.3 (~{WP}/IO_{2})
Other:
- note added: "BANK 0"
- note added: "BANK 1"
- note added: "BANK 2"
- note added: "BANK 3"
- note added: "BANK 6"
- note added: "BANK 7"
- note added: "BANK 8"
- note added: "CONFIG/JTAG"
- note added: "REMEMBER TO USE FOR JTAG PROG"
- note added: "SERDES DATA"
- note added: "SERDES PWR"
- note added: "TO DO THIS SHIT"

Commit message: Finished USB schematic, left pins for future work and worked on ESP32, FPGA config, things have been confirmed, next up is thinking about power and how it will function into if the system is going to be just a DVP camera or also MIPI
Parts:
- removed J1: Conn_02x03_Odd_Even, symbol Connector_Generic:Conn_02x03_Odd_Even
Connections:
- net FPGA_JTAG.~{FT_CTS} renamed FPGA_JTAG.CH_TDO
- net FPGA_JTAG.~{FT_DCD} renamed FPGA_JTAG.CH_TMS
- net FPGA_JTAG.~{FT_DSR} renamed FPGA_JTAG.CH_TCK
- net FPGA_JTAG.~{FT_RI} renamed FPGA_JTAG.CH_TDI
Other:
- note added: "THINGS I HAVE TO LINK"
- note added: "USB TO UART"
- note removed: "REMEMBER TO USE FOR JTAG PROG"
- note removed: "TO DO THIS SHIT"
- moved on the sheet: C1, R1, R10, R11, R12, R13, R14, R2, R3, R4, R5, R6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

Commit message: worked on power, should have external IC for sequencing and FPGA power is fine, started work in the CAMERA FPC, power 2V8 and 1V2 are there as LDOs, small package, should be fine.
Parts:
- removed R1, R2, R3, R4: 10K, PCM_JLCPCB:R_0402, symbol PCM_JLCPCB-Resistors:0402,10kΩ
- removed R11, R12, R13, R14: 4K7, PCM_JLCPCB:R_0402, symbol PCM_JLCPCB-Resistors:0402,4.7kΩ
- added RN1: 10K, PCM_Resistor_SMD_AKL:R_Array_Concave_4x0402, symbol PCM_Resistor_AKL:R_4x0402_Concave
- added RN2: 4K7, PCM_Resistor_SMD_AKL:R_Array_Concave_4x0402, symbol PCM_Resistor_AKL:R_4x0402_Concave
- renumbered R5 to R1, R6 to R2, R7 to R3, R8 to R4, R9 to R5, R10 to R6
Connections:
- net +3V3: now also RN1.5 (R4.2), RN1.6 (R3.2), RN1.7 (R2.2), RN1.8 (R1.2), RN2.6 (R3.2), RN2.7 (R2.2), RN2.8 (R1.2)
- net FLASH_MISO: now also RN1.3 (R3.1)
- net FLASH_MOSI: now also RN1.4 (R4.1)
- net FPGA_JTAG.CH_TCK: now also RN2.4 (R4.1)
- net FPGA_JTAG.CH_TDI: now also RN2.2 (R2.1)
- net FPGA_JTAG.CH_TDO: now also RN2.1 (R1.1)
- net FPGA_JTAG.CH_TMS: now also RN2.3 (R3.1)
- net GND: now also RN2.5 (R4.2)
- net ~{FLASH_RESET}: now also RN1.1 (R1.1)
- net ~{FLASH_WP}: now also RN1.2 (R2.1)
Other:
- moved on the sheet: U1I
