File: ecp5_sys_v1/USB.kicad_sch (KiCad schematic)
At the start: 0 parts

Commit message: Worked on USB
Parts:
- added C2, C3: 100n, PCM_JLCPCB:C_0402, symbol PCM_JLCPCB-Capacitors:0402,100nF
- added C4: 10u, PCM_JLCPCB:C_0603, symbol PCM_JLCPCB-Capacitors:0603,10uF
- added D1, D2: Yellow, PCM_JLCPCB:D_0603, symbol PCM_JLCPCB-Diodes:LED,0603,Yellow
- added D3: Red, PCM_JLCPCB:D_0603, symbol PCM_JLCPCB-Diodes:LED,0603,Red
- added F1: PTS060315V005, 1A, symbol Device:Polyfuse
- added FB1: (no value), PCM_JLCPCB:FB_0603, symbol PCM_JLCPCB-Inductors:Ferrite,0603,(2)
- added J2, J3: USB_C_Receptacle_USB2.0_16P, Connector_USB:USB_C_Receptacle_XKB_U262-16XN-4BVC11, symbol Connector:USB_C_Receptacle_USB2.0_16P
- added Q1: AO3401A, PCM_JLCPCB:Q_SOT-23, symbol PCM_JLCPCB-Transistors:PMOS,AO3401A
- added Q2, Q3: AO3400A, Package_TO_SOT_SMD:SOT-23, symbol Transistor_FET:AO3400A
- added R15, R16: 5K1, PCM_JLCPCB:R_0402, symbol PCM_JLCPCB-Resistors:0402,5.1kΩ
- added R17, R21: 100, PCM_JLCPCB:R_0402, symbol PCM_JLCPCB-Resistors:0402,100Ω
- added R18, R24, R25: 100K, PCM_JLCPCB:R_0402, symbol PCM_JLCPCB-Resistors:0402,100kΩ
- added R19, R20: 22, PCM_JLCPCB:R_0402, symbol PCM_JLCPCB-Resistors:0402,22Ω
- added R22: 1K5, PCM_JLCPCB:R_0402, symbol PCM_JLCPCB-Resistors:0402,1.5kΩ
- added R23: 4K7, PCM_JLCPCB:R_0402, symbol PCM_JLCPCB-Resistors:0402,4.7kΩ
- added R26: 330, PCM_JLCPCB:R_0402, symbol PCM_JLCPCB-Resistors:0402,150Ω
- added TP1: 5V_test, PCM_SparkFun-Connector:TestPoint-1.25mm, symbol Connector:TestPoint
- added U4: FT231XQ, Package_DFN_QFN:QFN-20-1EP_4x4mm_P0.5mm_EP2.5x2.5mm, symbol Interface_USB:FT231XQ
- added U5: USBLC6-2P6, Package_TO_SOT_SMD:SOT-666, symbol Power_Protection:USBLC6-2P6
Connections:
- new net: Q1.1 (G), R18.1
- new net: F1.2, FB1.1
- new net: R17.2, U4.14 (CBUS1)
- new net: R21.2, U4.7 (CBUS2)
- new net: Q2.3 (D), Q3.1 (G), R25.2
- new net: Q2.1 (G), R23.2, R24.1
- new net: Q3.2 (S), R26.1
- new net: D3.2, R26.2
- new net: R20.1, U5.6 (I/O1)
- new net: D2.1, R21.1
- new net: R19.2, U5.4 (I/O2)
- new net: D1.1, R17.1
- new net: J3.A4 (VBUS), J3.A9 (VBUS), J3.B4 (VBUS), J3.B9 (VBUS)
- new net 5V: Q1.2 (S), Q3.3 (D), R25.1, TP1.1, U4.12 (VCC)
- new net FT_3V3OUT: C2.1, D1.2, D2.2, U4.10 (3V3OUT), U4.11 (~{RESET}), U4.20 (VCCIO)
- new net FT_CBUS0: U4.15 (CBUS0)
- new net FT_CBUS3: U4.16 (CBUS3)
- new net FT_RXD: U4.1 (RXD)
- new net FT_TXD: U4.17 (TXD)
- new net GND: C2.2, C3.2, C4.2, D3.1, J2.A1 (GND), J2.A12 (GND), J2.B1 (GND), J2.B12 (GND), J2.SH (SHIELD), J3.A1 (GND), J3.A12 (GND), J3.B1 (GND), J3.B12 (GND), J3.SH (SHIELD), Q2.2 (S), R15.2, R16.2, R18.2, R24.2, U4.13 (GND), U4.21 (GND), U4.3 (GND), U5.2 (GND)
- new net LED_5V_TO: R23.1
- new net RAW_USB1_D+: J2.A6 (D+), J2.B6 (D+), U5.3 (I/O2)
- new net RAW_USB1_D-: J2.A7 (D-), J2.B7 (D-), U5.1 (I/O1)
- new net USB1_CC1: J2.A5 (CC1), R16.1
- new net USB1_CC2: J2.B5 (CC2), R15.1
- new net USB1_D-: R20.2, U4.9 (USBDM)
- new net USB1_PU: R22.2
- new net USB2_D+: R19.1, R22.1, U4.8 (USBDP)
- new net VBUS_NO_FILTER: C3.1, F1.1, J2.A4 (VBUS), J2.A9 (VBUS), J2.B4 (VBUS), J2.B9 (VBUS), U5.5 (VBUS)
- new net VBUS_PREMOS: C4.1, FB1.2, Q1.3 (D)
- new net ~{FT_CTS}: U4.6 (~{CTS})
- new net ~{FT_DCD}: U4.5 (~{DCD})
- new net ~{FT_DSR}: U4.4 (~{DSR})
- new net ~{FT_DTR}: U4.18 (~{DTR})
- new net ~{FT_RI}: U4.2 (~{RI})
- new net ~{FT_RTS}: U4.19 (~{RTS})
- no-connect marks 0 -> 2
Other:
- note added: "CLOSE TO FPGA"
- note added: "INIT 0V"
- note added: "LED PWR ON/OFF"
- note added: "USB TO UART/JTAG"
- note added: "USBC PROG"
- note added: "set to 3.3 to talk to a 3.3 device"

Commit message: Finished USB schematic, left pins for future work and worked on ESP32, FPGA config, things have been confirmed, next up is thinking about power and how it will function into if the system is going to be just a DVP camera or also MIPI
Parts:
- removed C2: 100n, PCM_JLCPCB:C_0402, symbol PCM_JLCPCB-Capacitors:0402,100nF
- removed D1, D2: Yellow, PCM_JLCPCB:D_0603, symbol PCM_JLCPCB-Diodes:LED,0603,Yellow
- removed F1: PTS060315V005, 1A, symbol Device:Polyfuse
- removed J3: USB_C_Receptacle_USB2.0_16P, Connector_USB:USB_C_Receptacle_XKB_U262-16XN-4BVC11, symbol Connector:USB_C_Receptacle_USB2.0_16P
- removed R17, R21: 100, PCM_JLCPCB:R_0402, symbol PCM_JLCPCB-Resistors:0402,100Ω
- removed R19, R20: 22, PCM_JLCPCB:R_0402, symbol PCM_JLCPCB-Resistors:0402,22Ω
- removed U4: FT231XQ, Package_DFN_QFN:QFN-20-1EP_4x4mm_P0.5mm_EP2.5x2.5mm, symbol Interface_USB:FT231XQ
- added C5, C6, C9: 100n, PCM_JLCPCB:C_0402, symbol PCM_JLCPCB-Capacitors:0402,100nF
- added C7, C8: 22p, PCM_JLCPCB:C_0402, symbol PCM_JLCPCB-Capacitors:0402,22pF
- added D4: Yellow, PCM_JLCPCB:D_0603, symbol PCM_JLCPCB-Diodes:LED,0603,Yellow
- added F3: SMD0805P075TF, 1.5A, EasyEDA:F0805, symbol EasyEDA:SMD0805P075TF
- added R19: 10K, PCM_JLCPCB:R_0402, symbol PCM_JLCPCB-Resistors:0402,10kΩ
- added R27: 100, PCM_JLCPCB:R_0402, symbol PCM_JLCPCB-Resistors:0402,100Ω
- added TP2: TestPoint, symbol Connector:TestPoint
- added U7: CH347F, EasyEDA:QFN-28_L4.0-W4.0-P0.40-BL-EP2.7, symbol EasyEDA:CH347F
- added X1: XL2EL89CSI-111YLC-8M, EasyEDA:CRYSTAL-SMD_4P-L3.2-W2.5-BL_SIT8008BI, symbol EasyEDA:XL2EL89CSI-111YLC-8M
- TP1: now not fitted
Connections:
- net USB2_D+ is gone; now on net CH_UD+: R22.1
- net GND: now also C5.2, C6.2, C7.2, C8.2, C9.2, U7.20 (GND), U7.29 (PAD), X1.2 (GND), X1.4 (GND)
- net VBUS_NO_FILTER: now also F3.1
- net at FB1.1: now also F3.2
- net CH_UD-: now reaches U5.6 (I/O1)
- net CH_UD-: now also U7.27 (UD-)
- net CH_UD+: now reaches U5.4 (I/O2)
- net CH_UD+: now also U7.28 (UD+)
- new net: D4.2, R27.1
- new net +3V3: C5.1, C6.1, R19.1, R27.2, U7.21 (VCC), U7.6 (VIO)
- new net CH_ACT: D4.1, U7.8 (ACT/SRST)
- new net CH_DTR0: U7.10 (DTR0/TNOW0/GPIO2)
- new net CH_RST0: U7.18 (RTS0/GPIO1)
- new net CH_RXD0: U7.22 (RXD0)
- new net CH_RXD1: U7.5 (RXD1)
- new net CH_TCK: U7.23 (TCK/SWDCLK/GPIO4)
- new net CH_TDI: U7.25 (TDI/GPIO6)
- new net CH_TDO: U7.24 (TDO/GPIO5)
- new net CH_TMS: U7.26 (TMS/SWDIO/GPIO7)
- new net CH_TXD0: U7.19 (TXD0)
- new net CH_TXD1: U7.4 (TXD1)
- new net CH_XD: C8.1, U7.2 (XO), X1.3
- new net CH_XI: C7.1, U7.1 (XI), X1.1
- new net CH_~{RST}: C9.1, R19.2, TP2.1, U7.3 (~{RST})
- no-connect marks 2 -> 11
Other:
- note added: "1ms"
- note added: "ESP"
- note added: "FPGA"
- note added: "PTS060315V005, 1A"
- note removed: "set to 3.3 to talk to a 3.3 device"

Commit message: worked on power, should have external IC for sequencing and FPGA power is fine, started work in the CAMERA FPC, power 2V8 and 1V2 are there as LDOs, small package, should be fine.
Parts:
- TP4: renamed from TP1; value 5V_test -> +5V_test
- renumbered C5 to C28, C6 to C29, C3 to C30, C4 to C31, C7 to C32, C9 to C33, C8 to C34, D4 to D1, D3 to D2, F3 to F1, J2 to J1, Q1 to Q2, Q2 to Q3, Q3 to Q4, R15 to R19, R16 to R20, R27 to R21, R18 to R22, R22 to R23, R23 to R24, R24 to R25, R19 to R26, R25 to R27, R26 to R28, TP2 to TP5, U7 to U10, U5 to U11
Connections:
- net 5V renamed +5V
